File: KiCad/ServoTester/ServoTester.sch (KiCad schematic (older format))
At the start: 14 parts, among them J1 WiiNunchuckConnector, J2 Conn_01x02_Female, M1 Motor_Servo_JR, M2 Motor_Servo_JR, M3 Motor_Servo_JR, M4 Motor_Servo_JR, U1 Teensy2.0, U2 HD44780

Commit message: working on board
Parts:
- J1: footprint (none) -> ServoTester:WiiNunchuckConnector
- U2: footprint (none) -> ServoTester:JHD204AO 20x4 Character LCD
Changed lines of the file:
@@
 EESchema Schematic File Version 4
+LIBS:ServoTester-cache
 EELAYER 26 0
 EELAYER END
@@
 F 0 "J1" H 5477 1596 50  0000 L CNN
 F 1 "WiiNunchuckConnector" H 5477 1505 50  0000 L CNN
-F 2 "" H 5050 1900 50  0001 C CNN
+F 2 "ServoTester:WiiNunchuckConnector" H 5050 1900 50  0001 C CNN
 F 3 "" H 5050 1900 50  0001 C CNN
 	1    5200 1600
@@
 F 0 "U2" H 4278 4882 50  0000 L CNN
 F 1 "HD44780" H 4278 4791 50  0000 L CNN
-F 2 "" H 2600 4500 50  0001 C CNN
+F 2 "ServoTester:JHD204AO 20x4 Character LCD" H 2600 4500 50  0001 C CNN
 F 3 "" H 2600 4500 50  0001 C CNN
 	1    3400 4800

Commit message: think board is ready for prototyping
Parts:
- added C1: CP1, Capacitor_THT:CP_Radial_D8.0mm_P5.00mm, symbol Device:CP1
- added R2: R_US, Resistor_THT:R_Axial_DIN0207_L6.3mm_D2.5mm_P10.16mm_Horizontal, symbol Device:R_US
- added SW1: SW_Push_Open, Button_Switch_THT:SW_PUSH_6mm_H5mm, symbol Switch:SW_Push_Open
- RV1: footprint Connector_Wire:SolderWirePad_1x03_P3.175mm_Drill1mm -> ServoTester:Potentiometer
Connections:
- net GND: now also C1.2, SW1.1 (A)
- net VCC: now also C1.1, R2.1
- net at U1.2 (0): now also R2.2, SW1.2 (B)
- net at U1.23 (16_A5): now also U2.6 (E); no longer U2.4 (RS)
- net at U1.24 (17_A4): now also U2.4 (RS); no longer U2.6 (E)
Changed lines of the file:
@@
 F 0 "RV1" H 2482 3896 50  0000 R CNN
 F 1 "10k" H 2482 3805 50  0000 R CNN
-F 2 "Connector_Wire:SolderWirePad_1x03_P3.175mm_Drill1mm" H 2550 3850 50  0001 C CNN
+F 2 "ServoTester:Potentiometer" H 2550 3850 50  0001 C CNN
 F 3 "~" H 2550 3850 50  0001 C CNN
 	1    2550 3850
@@
 	3650 4150 3650 4450
 Wire Wire Line
-	3650 2400 3700 2400
-Wire Wire Line
-	3700 2400 3700 4100
-Wire Wire Line
 	3700 4100 3150 4100
 Wire Wire Line
@@
 	3600 2500 3650 2500
 Wire Wire Line
-	4250 2500 4250 3650
-Wire Wire Line
 	4250 3650 2950 3650
 Wire Wire Line
 	2950 3650 2950 4450
-Connection ~ 3650 2500
-Wire Wire Line
-	3650 2500 4250 2500
 $Comp
 L Connector:Conn_01x02_Female J2
@@
 Wire Wire Line
 	8200 3600 8950 3600
+$Comp
+L Device:CP1 C1
+U 1 1 5D2A2AFF
+P 5600 3100
+F 0 "C1" H 5715 3146 50  0000 L CNN
+F 1 "CP1" H 5715 3055 50  0000 L CNN
+F 2 "Capacitor_THT:CP_Radial_D8.0mm_P5.00mm" H 5600 3100 50  0001 C CNN
+F 3 "~" H 5600 3100 50  0001 C CNN
+	1    5600 3100
+	1    0    0    -1
+$EndComp
+Wire Wire Line
+	5600 2950 5600 2900
+Wire Wire Line
+	5600 2900 6100 2900
+Connection ~ 6100 2900
+Wire Wire Line
+	5600 3250 5600 3600
+Connection ~ 5600 3600
+Wire Wire Line
+	2250 1700 1950 1700
+$Comp
+L Device:R_US R2
+U 1 1 5D2B0146
+P 1950 1350
+F 0 "R2" H 2018 1396 50  0000 L CNN
+F 1 "R_US" H 2018 1305 50  0000 L CNN
+F 2 "Resistor_THT:R_Axial_DIN0207_L6.3mm_D2.5mm_P10.16mm_Horizontal" V 1990 1340 50  0001 C CNN
+F 3 "~" H 1950 1350 50  0001 C CNN
+	1    1950 1350
+	1    0    0    -1
+$EndComp
+$Comp
+L power:VCC #PWR0115
+U 1 1 5D2B0293
+P 1950 1100
+F 0 "#PWR0115" H 1950 950 50  0001 C CNN
+F 1 "VCC" H 1967 1273 50  0000 C CNN
+F 2 "" H 1950 1100 50  0001 C CNN
+F 3 "" H 1950 1100 50  0001 C CNN
+	1    1950 1100
+	1    0    0    -1
+$EndComp
+$Comp
+L power:GND #PWR0116
+U 1 1 5D2B37F4
+P 1400 1850
+F 0 "#PWR0116" H 1400 1600 50  0001 C CNN
+F 1 "GND" H 1405 1677 50  0000 C CNN
+F 2 "" H 1400 1850 50  0001 C CNN
+F 3 "" H 1400 1850 50  0001 C CNN
+	1    1400 1850
+	1    0    0    -1
+$EndComp
+Wire Wire Line
+	1950 1500 1950 1700
+Connection ~ 1950 1700
+Wire Wire Line
+	1950 1700 1800 1700
+Wire Wire Line
+	1950 1200 1950 1100
+Wire Wire Line
+	1400 1700 1400 1850
+$Comp
+L Switch:SW_Push_Open SW1
+U 1 1 5D2BF127
+P 1600 1700
+F 0 "SW1" H 1600 1915 50  0000 C CNN
+F 1 "SW_Push_Open" H 1600 1824 50  0000 C CNN
+F 2 "Button_Switch_THT:SW_PUSH_6mm_H5mm" H 1600 1900 50  0001 C CNN
+F 3 "" H 1600 1900 50  0001 C CNN
+	1    1600 1700
+	1    0    0    -1
+$EndComp
+Wire Wire Line
+	4250 2400 4250 3650
+Wire Wire Line
+	3650 2400 4250 2400
+Wire Wire Line
+	3650 2500 3700 2500
+Wire Wire Line
+	3700 2500 3700 4100
+Connection ~ 3650 2500
 $EndSCHEMATC

Commit message: fixing board
Parts:
- J2: footprint Connector:Banana_Jack_2Pin -> ServoTester:BananaJack_2
- JP1, JP2, JP3, JP4, M1, M2, M3, M4: footprint Connector_Wire:SolderWirePad_1x03_P3.175mm_Drill1mm -> Connector_PinHeader_2.54mm:PinHeader_1x03_P2.54mm_Vertical
Changed lines of the file:
@@
 F 0 "JP1" V 6054 3317 50  0000 L CNN
 F 1 "Jumper_3_Bridged12" V 6145 3317 50  0000 L CNN
-F 2 "Connector_Wire:SolderWirePad_1x03_P3.175mm_Drill1mm" H 6100 3250 50  0001 C CNN
+F 2 "Connector_PinHeader_2.54mm:PinHeader_1x03_P2.54mm_Vertical" H 6100 3250 50  0001 C CNN
 F 3 "~" H 6100 3250 50  0001 C CNN
 	1    6100 3250
@@
 F 0 "JP2" V 6554 3317 50  0000 L CNN
 F 1 "Jumper_3_Bridged12" V 6645 3317 50  0000 L CNN
-F 2 "Connector_Wire:SolderWirePad_1x03_P3.175mm_Drill1mm" H 6600 3250 50  0001 C CNN
+F 2 "Connector_PinHeader_2.54mm:PinHeader_1x03_P2.54mm_Vertical" H 6600 3250 50  0001 C CNN
 F 3 "~" H 6600 3250 50  0001 C CNN
 	1    6600 3250
@@
 F 0 "JP3" V 7054 3317 50  0000 L CNN
 F 1 "Jumper_3_Bridged12" V 7145 3317 50  0000 L CNN
-F 2 "Connector_Wire:SolderWirePad_1x03_P3.175mm_Drill1mm" H 7100 3250 50  0001 C CNN
+F 2 "Connector_PinHeader_2.54mm:PinHeader_1x03_P2.54mm_Vertical" H 7100 3250 50  0001 C CNN
 F 3 "~" H 7100 3250 50  0001 C CNN
 	1    7100 3250
@@
 F 0 "JP4" V 7554 3317 50  0000 L CNN
 F 1 "Jumper_3_Bridged12" V 7645 3317 50  0000 L CNN
-F 2 "Connector_Wire:SolderWirePad_1x03_P3.175mm_Drill1mm" H 7600 3250 50  0001 C CNN
+F 2 "Connector_PinHeader_2.54mm:PinHeader_1x03_P2.54mm_Vertical" H 7600 3250 50  0001 C CNN
 F 3 "~" H 7600 3250 50  0001 C CNN
 	1    7600 3250
@@
 F 0 "M2" V 6399 4206 50  0000 L CNN
 F 1 "Motor_Servo_JR" V 6490 4206 50  0000 L CNN
-F 2 "Connector_Wire:SolderWirePad_1x03_P3.175mm_Drill1mm" H 6450 3810 50  0001 C CNN
+F 2 "Connector_PinHeader_2.54mm:PinHeader_1x03_P2.54mm_Vertical" H 6450 3810 50  0001 C CNN
 F 3 "http://forums.parallax.com/uploads/attachments/46831/74481.png" H 6450 3810 50  0001 C CNN
 	1    6450 4000
@@
 F 0 "M1" V 5899 4206 50  0000 L CNN
 F 1 "Motor_Servo_JR" V 5990 4206 50  0000 L CNN
-F 2 "Connector_Wire:SolderWirePad_1x03_P3.175mm_Drill1mm" H 5950 3810 50  0001 C CNN
+F 2 "Connector_PinHeader_2.54mm:PinHeader_1x03_P2.54mm_Vertical" H 5950 3810 50  0001 C CNN
 F 3 "http://forums.parallax.com/uploads/attachments/46831/74481.png" H 5950 3810 50  0001 C CNN
 	1    5950 4000
@@
 F 0 "M3" V 6899 4206 50  0000 L CNN
 F 1 "Motor_Servo_JR" V 6990 4206 50  0000 L CNN
-F 2 "Connector_Wire:SolderWirePad_1x03_P3.175mm_Drill1mm" H 6950 3810 50  0001 C CNN
+F 2 "Connector_PinHeader_2.54mm:PinHeader_1x03_P2.54mm_Vertical" H 6950 3810 50  0001 C CNN
 F 3 "http://forums.parallax.com/uploads/attachments/46831/74481.png" H 6950 3810 50  0001 C CNN
 	1    6950 4000
@@
 F 0 "M4" V 7399 4206 50  0000 L CNN
 F 1 "Motor_Servo_JR" V 7490 4206 50  0000 L CNN
-F 2 "Connector_Wire:SolderWirePad_1x03_P3.175mm_Drill1mm" H 7450 3810 50  0001 C CNN
+F 2 "Connector_PinHeader_2.54mm:PinHeader_1x03_P2.54mm_Vertical" H 7450 3810 50  0001 C CNN
 F 3 "http://forums.parallax.com/uploads/attachments/46831/74481.png" H 7450 3810 50  0001 C CNN
 	1    7450 4000
@@
 F 0 "J2" H 9177 3476 50  0000 L CNN
 F 1 "Conn_01x02_Female" H 9177 3385 50  0000 L CNN
-F 2 "Connector:Banana_Jack_2Pin" H 9150 3500 50  0001 C CNN
+F 2 "ServoTester:BananaJack_2" H 9150 3500 50  0001 C CNN
 F 3 "~" H 9150 3500 50  0001 C CNN
 	1    9150 3500
